File: climbingRGB.brd (EAGLE design)
At the start: 31.8 x 15.9 mm, 3 parts

Commit message: minor edits
- changed RGB board hole to 7/16"
- minor edits to MCU board
Parts:
- moved LED4 0.25 mm to (8.64, 7.62)
- moved LED3 0.25 mm to (28.2, 7.62)
Routing:
- net N$5: track 15.2 -> 16.3 mm
- net N$6: track 15.1 -> 15.6 mm
Other:
- board text added: "v1.3 - 7/16 hole"
- board text removed: "v1.2"
