File: control_board_MCU.sch (EAGLE design)
At the start: 49 parts, among them U1 ATMEGA168, U2 ###V, Y1 16MHZ

Commit message: minor edits
- changed RGB board hole to 7/16"
- minor edits to MCU board
Parts:
- removed C10: 0.1uF, SparkFun:CAP0402
- removed R11: 10K, SparkFun:RESISTOR0402
- removed R7, R8, R9: 4.7k, SparkFun-Passives:RESISTOR0402-RES
- removed U$19: RJ45-8PTH, SparkFun-Connectors:RJ45-8PTH
- added C6: 0.1uF, SparkFun-Capacitors:CAP0402-CAP
- added F1: (no value), adafruit:PTCFUSE-1812
- added LED2: Red, SparkFun:LED0603
- LED1: value Red -> Blue
- R1, R2: value 1.8k -> 2.7k
- R3: device SparkFun-Passives:RESISTOR0603-RES -> SparkFun-Passives:RESISTOR0402-RES
- R4: device SparkFun-Passives:RESISTOR0402-RES -> SparkFun-Passives:RESISTOR1206
- R5: value 100 -> 1k; device SparkFun-Passives:RESISTOR0402-RES -> SparkFun:RESISTOR0402
- R6: value 4.7k -> 1k; device SparkFun-Passives:RESISTOR0402-RES -> SparkFun:RESISTOR0402
- renumbered C13 to C7, C19 to C8, STANDOFF4 to STANDOFF1, TLC1 to TLC5947-2, U2 to MIC5205
Connections:
- removed net N$9: R9.1, U$21.1
- net DATA2+: no longer R5.1
- net DATA2-: now also U$18.6; no longer R5.2, U$18.4
- net GND: now also C6.2, U$21.1, U$21.2, U$21.3, U$21.4, U1.ADC7, U1.PB0(ICP), U1.PC4(ADC4/SDA), U1.PC5(ADC5/SCL), U1.PD3(INT1), U1.PD4(XCK/T0), U1.PD5(T1), U1.PD6(AIN0), U1.PD7(AIN1); no longer C10.2
- net N$38: now also R6.1; no longer R11.1
- net N$6: now also LED2.C, U1.ADC6; no longer R6.1, U$21.4
- net N$7: now also LED2.A, R5.1; no longer R7.1, U$21.3
- net N$8: now also F1.1, JP1.1; no longer R8.1, U$21.2
- net NC: now also U$18.4; no longer U$18.6
- net VCC: now also C6.1, R5.2; no longer C10.1, R11.2, R7.2, R8.2, R9.2
- net VDD: now also F1.2; no longer JP1.1
Other:
- moved on the sheet: R5, R6, U$18
