File: climbing_WS2812.sch (EAGLE design)
At the start: 8 parts

Commit message: new things!
Connections:
- new net N$2: U$1.1, U$3.DO
Changed lines of the file:
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@@
+</segment>
+</net>
+<net name="N$2" class="0">
+<segment>
+<pinref part="U$3" gate="G$1" pin="DO"/>
+<wire x1="53.34" y1="86.36" x2="53.34" y2="53.34" width="0.1524" layer="91"/>
+<pinref part="U$1" gate="G$1" pin="1"/>
+<wire x1="53.34" y1="53.34" x2="-15.24" y2="53.34" width="0.1524" layer="91"/>
 </segment>
 </net>
