File: control_board_MCU.brd (EAGLE design)
At the start: 80 x 35.6 mm, 50 parts, among them U1 ATMEGA168, U2 ###V, Y1 16MHZ

Commit message: minor edits
- changed RGB board hole to 7/16"
- minor edits to MCU board
Parts:
- removed C10: 0.1uF, SparkFun:C0402
- removed C19: 10uF, SparkFun:EIA3216
- removed R11: 10K, SparkFun:C0402
- removed R7, R8, R9: 4.7k, SparkFun-Passives:0402-RES
- removed U$19: RJ45-8PTH, SparkFun-Connectors:RJ45-8
- added C6: 0.1uF, SparkFun-Capacitors:0402-CAP
- added C8: 10uF, SparkFun:EIA3216
- added F1: (no value), adafruit:1812
- added LED2: Red, SparkFun:LED-0603
- added STANDOFF1, STANDOFF3: STAND-OFF, SparkFun-Electromechanical:STAND-OFF
- LED1: value Red -> Blue
- R1, R2: value 1.8k -> 2.7k
- R3: device SparkFun-Passives:0603-RES -> SparkFun-Passives:0402-RES
- R4: device SparkFun-Passives:0402-RES -> SparkFun-Passives:1206
- R5: value 100 -> 1k; device SparkFun-Passives:0402-RES -> SparkFun:C0402
- R6: value 4.7k -> 1k; device SparkFun-Passives:0402-RES -> SparkFun:C0402
- moved JP1 55.0 mm to (77.6, 17.8), turned to 270 degrees
- moved R5 25.9 mm to (42.9, 17.7)
- moved STANDOFF4 13.1 mm to (78.7, 11.3)
- moved R6 7.50 mm to (17.5, 24.1), turned to 225 degrees
- moved R4 1.55 mm to (18.1, 19.0)
- moved LED1 1.37 mm to (18.7, 23.0), turned to 135 degrees
- moved STANDOFF2 1.30 mm to (7.62, 33.0)
- moved JP4 0.38 mm to (13.5, 33.7)
- renumbered C13 to C7, TLC1 to TLC5947-2, U2 to MIC5205
Connections:
- removed net N$9: R9.1, U$21.1
- net DATA2+: no longer R5.1
- net DATA2-: now also U$18.6; no longer R5.2, U$18.4
- net GND: now also C6.2, C8.C, U$21.1, U$21.2, U$21.3, U$21.4, U1.1, U1.10, U1.11, U1.12, U1.2, U1.22, U1.27, U1.28, U1.9; no longer C10.2, C19.C
- net N$38: now also R6.1; no longer R11.1
- net N$6: now also LED2.C, U1.19; no longer R6.1, U$21.4
- net N$7: now also LED2.A, R5.1; no longer R7.1, U$21.3
- net N$8: now also F1.1, JP1.2; no longer R8.1, U$21.2
- net NC: now also U$18.4; no longer U$18.6
- net VCC: now also C6.1, R5.2; no longer C10.1, R11.2, R7.2, R8.2, R9.2
- net VDD: now also C8.A, F1.2; no longer C19.A, JP1.2
Routing:
- net GND: track 50.3 -> 76.3 mm, vias 13 -> 15
- net VDD: track 168.5 -> 177.1 mm
- net VCC: track 110.0 -> 102.8 mm
- net DATA2+: track 4.58 -> 0.00 mm
- net N$8: track 1.90 -> 4.00 mm
- net DATA2-: track 2.04 -> 0.00 mm
- net N$9: track 1.90 -> 0.00 mm
- net BLANK: track 60.1 -> 58.3 mm
- net DATA1+: track 10.2 -> 11.9 mm
- net N$6: track 1.90 -> 3.00 mm
- net N$38: track 2.39 -> 1.66 mm
- net XLAT: track 76.6 -> 76.0 mm
Other:
- board size 80 x 35.6 mm -> 77.5 x 35.6 mm
- board text added: "1 2 3 4 5 6 7 8"
- board text added: "16 15 14 13 12 11 10 9"
- board text added: "RST SCK MISO GND MOSI VCC"
- board text removed: "0, 1, 2"
- board text removed: "12, 13, 14"
- board text removed: "15, 16, 17"
- board text removed: "18, 19, 20"
- board text removed: "21, 22, 23"
- board text removed: "3, 4, 5"
- board text removed: "6, 7, 8"
- board text removed: "9, 10, 11"

Commit message: new things!
Parts:
- removed JP1: (no value), SparkFun-Connectors:JST-2-SMD
- removed STANDOFF3: STAND-OFF, SparkFun-Electromechanical:STAND-OFF
- removed U$1, U$10, U$11, U$12, U$13, U$14, U$15, U$16, U$2, U$3, U$4, U$5, U$6, U$7, U$8, U$9: SWR204-D02, SparkFun-Connectors:SWR204
- added 1, 10, 11, 12, 13, 14, 15, 16, 2, 3, 4, 5, 6, 7, 8, 9: (no value), pinhead:2X02
- added C9: 100uF, SparkFun-Capacitors:PANASONIC_C
- added J1: POWER_JACKPTH, SparkFun-Connectors:POWER_JACK_PTH
- moved F1 51.2 mm to (18.3, 4.57), turned to 270 degrees
- moved STANDOFF1 50.4 mm to (28.6, 30.7)
- moved STANDOFF2 31.3 mm to (14.1, 2.41)
- moved R5 21.6 mm to (21.7, 13.3)
- moved LED2 18.6 mm to (22.7, 15.6), turned to 270 degrees
- moved STANDOFF4 12.6 mm to (89.2, 18.4)
- moved U$18 10.7 mm to (2.92, 18.2)
- moved U$21 8.46 mm to (6.48, 32.0)
- moved C1 7.73 mm to (66.9, 18.9)
- moved R1 7.73 mm to (69.2, 18.0)
- moved R2 7.73 mm to (55.9, 20.8)
- moved TLC5947 7.73 mm to (62.5, 12.7)
- moved TLC5947-2 7.73 mm to (62.5, 25.4)
- moved C2 7.73 mm to (58.2, 19.3)
- moved MIC5205 5.91 mm to (16.0, 12.1), turned to 270 degrees
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Connections:
- removed net OUT1: TLC5947.6, U$1.P$2
- removed net OUT2: TLC5947.7, U$1.P$1
- new net N$14: 1.2, TLC5947.6
- new net N$9: 1.1, TLC5947.7
- net GND: now also C9.-, J1.GND, J1.GNDBREAK, U1.19; no longer JP1.1, U1.1
- net N$6: now also U1.1; no longer U1.19
- net N$8: now also J1.PWR; no longer JP1.2
- net OUT0: now also 1.3; no longer U$1.P$3
- net OUT10: now also 4.2; no longer U$4.P$2
- net OUT11: now also 4.1; no longer U$4.P$1
- net OUT12: now also 5.3; no longer U$5.P$3
- net OUT13: now also 5.2; no longer U$5.P$2
- net OUT14: now also 5.1; no longer U$5.P$1
- net OUT15: now also 6.3; no longer U$6.P$3
- net OUT16: now also 6.2; no longer U$6.P$2
- net OUT17: now also 6.1; no longer U$6.P$1
- net OUT18: now also 7.3; no longer U$7.P$3
- net OUT19: now also 7.2; no longer U$7.P$2
- net OUT20: now also 7.1; no longer U$7.P$1
- net OUT21: now also 8.3; no longer U$8.P$3
- net OUT22: now also 8.2; no longer U$8.P$2
- net OUT23: now also 8.1; no longer U$8.P$1
- net OUT24: now also 9.3; no longer U$9.P$3
- net OUT25: now also 9.2; no longer U$9.P$2
- net OUT26: now also 9.1; no longer U$9.P$1
- net OUT27: now also 10.3; no longer U$10.P$3
- net OUT28: now also 10.2; no longer U$10.P$2
- net OUT29: now also 10.1; no longer U$10.P$1
- net OUT3: now also 2.3; no longer U$3.P$3
- net OUT30: now also 11.3; no longer U$11.P$3
- net OUT31: now also 11.2; no longer U$11.P$2
- net OUT32: now also 11.1; no longer U$11.P$1
- net OUT33: now also 12.3; no longer U$12.P$3
- net OUT34: now also 12.2; no longer U$12.P$2
- net OUT35: now also 12.1; no longer U$12.P$1
- net OUT36: now also 13.3; no longer U$13.P$3
- net OUT37: now also 13.2; no longer U$13.P$2
- net OUT38: now also 13.1; no longer U$13.P$1
- net OUT39: now also 14.3; no longer U$14.P$3
- net OUT4: now also 2.2; no longer U$3.P$2
- net OUT40: now also 14.2; no longer U$14.P$2
- net OUT41: now also 14.1; no longer U$14.P$1
- net OUT42: now also 15.3; no longer U$15.P$3
- net OUT43: now also 15.2; no longer U$15.P$2
- net OUT44: now also 15.1; no longer U$15.P$1
- net OUT45: now also 16.3; no longer U$16.P$3
- net OUT46: now also 16.2; no longer U$16.P$2
- net OUT47: now also 16.1; no longer U$16.P$1
- net OUT5: now also 2.1; no longer U$3.P$1
- net OUT6: now also 3.3; no longer U$2.P$3
- net OUT7: now also 3.2; no longer U$2.P$2
- net OUT8: now also 3.1; no longer U$2.P$1
- net OUT9: now also 4.3; no longer U$4.P$3
- net VDD: now also 1.4, 10.4, 11.4, 12.4, 13.4, 14.4, 15.4, 16.4, 2.4, 3.4, 4.4, 5.4, 6.4, 7.4, 8.4, 9.4, C9.+; no longer U$1.P$4, U$10.P$4, U$11.P$4, U$12.P$4, U$13.P$4, U$14.P$4, U$15.P$4, U$16.P$4, U$2.P$4, U$3.P$4, U$4.P$4, U$5.P$4, U$6.P$4, U$7.P$4, U$8.P$4, U$9.P$4
Routing:
- net N$9: track 0.00 -> 36.0 mm
- net VCC: track 102.8 -> 138.5 mm, vias 4 -> 2
- net N$14: track 0.00 -> 35.2 mm
- net VDD: track 177.1 -> 207.7 mm, vias 0 -> 1
- net OUT2: track 22.4 -> 0.00 mm
- net OUT1: track 21.9 -> 0.00 mm
- net SCLK: track 69.7 -> 89.6 mm
- net OUT0: track 24.2 -> 38.0 mm
- net SIN: track 27.7 -> 38.9 mm
- net OUT44: track 21.5 -> 32.4 mm
- net SOUT1: track 30.6 -> 41.0 mm
- net XLAT: track 76.0 -> 86.1 mm
- net BLANK: track 58.3 -> 68.4 mm
- net OUT43: track 16.7 -> 26.8 mm
- net OUT3: track 17.0 -> 27.0 mm
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Other:
- board size 77.5 x 35.6 mm -> 92.7 x 38.1 mm
- board text added: "v1.5"
- board text removed: "1 2 3 4 5 6 7 8"
- board text removed: "16 15 14 13 12 11 10 9"
- board text removed: "VDD GND"
- board text removed: "v1.4"
