File: control_board_WS2812.sch (EAGLE design)
At the start: 47 parts, among them J1 POWER_JACKPTH, U1 ATMEGA168, Y1 16MHZ

Commit message: new things!
Parts:
- removed 1, 10, 11, 12, 13, 14, 15, 16, 2, 3, 4, 5, 6, 7, 8, 9: (no value), pinhead:PINHD-2X2
- removed R1, R2: 2.7k, SparkFun-Resistors:RESISTOR0603-RES
- removed TLC5947, TLC5947-2: TLC5947DAP, SparkFun-DigitalIC:TLC5947DAP
- added JP1, JP10, JP11, JP12, JP13, JP14, JP15, JP16, JP2, JP3, JP5, JP6, JP7, JP8, JP9: (no value), pinhead:PINHD-2X2
- added U$1, U$2: M74HC238TSSOP16, SparkFun-DigitalIC:M74HC238TSSOP16
- added U$3: INVERTING_SCHMITT_TRIGGER, SparkFun-DigitalIC:INVERTING_SCHMITT_TRIGGER
- C2: value .1uF -> (none); device SparkFun-Capacitors:CAP0402-CAP -> SparkFun-Capacitors:CAP_POLC
- C9: value 100uF -> .1uF; device SparkFun-Capacitors:CAP_POLC -> SparkFun-Capacitors:CAP0402-CAP
- JP4: device SparkFun-Connectors:M06LOCK -> pinhead:PINHD-2X2
Connections:
- removed net BLANK: JP4.4, TLC5947-2.BLANK, TLC5947.BLANK, U1.PB2(SS/OC1B)
- removed net N$10: U$21.5, U1.PC0(ADC0)
- removed net N$11: U$21.6, U1.PC1(ADC1)
- removed net N$12: U$21.7, U1.PC2(ADC2)
- removed net N$13: U$21.8, U1.PC3(ADC3)
- removed net N$6: LED2.C, U1.PD3(INT1)
- removed net OUT0: 1.3, TLC5947.OUT0
- removed net OUT10: 4.2, TLC5947.OUT10
- removed net OUT11: 4.1, TLC5947.OUT11
- removed net OUT12: 5.3, TLC5947.OUT12
- removed net OUT13: 5.2, TLC5947.OUT13
- removed net OUT14: 5.1, TLC5947.OUT14
- removed net OUT15: 6.3, TLC5947.OUT15
- removed net OUT16: 6.2, TLC5947.OUT16
- removed net OUT17: 6.1, TLC5947.OUT17
- removed net OUT18: 7.3, TLC5947.OUT18
- removed net OUT19: 7.2, TLC5947.OUT19
- removed net OUT20: 7.1, TLC5947.OUT20
- removed net OUT21: 8.3, TLC5947.OUT21
- removed net OUT22: 8.2, TLC5947.OUT22
- removed net OUT23: 8.1, TLC5947.OUT23
- removed net OUT24: 9.3, TLC5947-2.OUT0
- removed net OUT25: 9.2, TLC5947-2.OUT1
- removed net OUT26: 9.1, TLC5947-2.OUT2
- removed net OUT27: 10.3, TLC5947-2.OUT3
- removed net OUT28: 10.2, TLC5947-2.OUT4
- removed net OUT29: 10.1, TLC5947-2.OUT5
- removed net OUT3: 2.3, TLC5947.OUT3
- removed net OUT30: 11.3, TLC5947-2.OUT6
- removed net OUT31: 11.2, TLC5947-2.OUT7
- removed net OUT32: 11.1, TLC5947-2.OUT8
- removed net OUT33: 12.3, TLC5947-2.OUT9
- removed net OUT34: 12.2, TLC5947-2.OUT10
- removed net OUT35: 12.1, TLC5947-2.OUT11
- removed net OUT36: 13.3, TLC5947-2.OUT12
- removed net OUT37: 13.2, TLC5947-2.OUT13
- removed net OUT38: 13.1, TLC5947-2.OUT14
- removed net OUT39: 14.3, TLC5947-2.OUT15
- removed net OUT4: 2.2, TLC5947.OUT4
- removed net OUT40: 14.2, TLC5947-2.OUT16
- removed net OUT41: 14.1, TLC5947-2.OUT17
- removed net OUT42: 15.3, TLC5947-2.OUT18
- removed net OUT43: 15.2, TLC5947-2.OUT19
- removed net OUT44: 15.1, TLC5947-2.OUT20
- removed net OUT45: 16.3, TLC5947-2.OUT21
- removed net OUT46: 16.2, TLC5947-2.OUT22
- removed net OUT47: 16.1, TLC5947-2.OUT23
- removed net OUT5: 2.1, TLC5947.OUT5
- removed net OUT6: 3.3, TLC5947.OUT6
- removed net OUT7: 3.2, TLC5947.OUT7
- removed net OUT8: 3.1, TLC5947.OUT8
- removed net OUT9: 4.3, TLC5947.OUT9
- removed net SCLK: JP4.5, TLC5947-2.SCLK, TLC5947.SCLK, U$20.SCK, U1.PB5(SCK)
- removed net SIN: TLC5947.SIN, U$20.MOSI, U1.PB3(MOSI/OC2)
- removed net SOUT: TLC5947-2.SIN, TLC5947.SOUT
- removed net SOUT1: JP4.6, TLC5947-2.SOUT
- removed net XLAT: JP4.3, TLC5947-2.XLAT, TLC5947.XLAT, U1.PB1(OC1A)
- new net /G2B: U$1.~G2B, U$3.A, U1.PC3(ADC3)
- new net 10: U$21.7, U1.PD6(AIN0)
- new net 11: U$21.6, U1.PD7(AIN1)
- new net 12: U$21.5, U1.PB0(ICP)
- new net 9: U$21.8, U1.PD5(T1)
- new net A: U$1.A, U$2.A, U1.PC0(ADC0)
- new net B: U$1.B, U$2.B, U1.PC1(ADC1)
- new net C: U$1.C, U$2.C, U1.PC2(ADC2)
- new net G2B: U$2.~G2B, U$3.Y
- new net MOSI: U$20.MOSI, U1.PB3(MOSI/OC2)
- new net N$15: JP5.1
- new net N$16: JP6.1
- new net N$17: JP7.1
- new net N$18: JP8.1
- new net N$19: JP9.1
- new net N$20: JP10.1
- new net N$21: JP11.1
- new net N$22: JP12.1
- new net N$23: JP13.1
- new net N$24: JP14.1
- new net N$25: JP15.1
- new net N$26: JP16.1
- new net NC1: U$18.5
- new net SCK: LED2.C, U$20.SCK, U1.PB5(SCK)
- new net WS: U$1.G1, U$2.G1, U1.PB1(OC1A)
- new net Y0-1: JP8.3, U$1.Y0
- new net Y0-2: JP16.3, U$2.Y0
- new net Y1-1: JP7.3, U$1.Y1
- new net Y1-2: JP15.3, U$2.Y1
- new net Y2-1: JP6.3, U$1.Y2
- new net Y2-2: JP14.3, U$2.Y2
- new net Y3-1: JP5.3, U$1.Y3
- new net Y3-2: JP13.3, U$2.Y3
- new net Y4-1: JP4.3, U$1.Y4
- new net Y4-2: JP12.3, U$2.Y4
- new net Y5-1: JP3.3, U$1.Y5
- new net Y5-2: JP11.3, U$2.Y5
- new net Y6-1: JP2.3, U$1.Y6
- new net Y6-2: JP10.3, U$2.Y6
- new net Y7-1: JP1.3, U$1.Y7
- new net Y7-2: JP9.3, U$2.Y7
- net GND: now also C2.-, C9.2, JP1.2, JP10.2, JP11.2, JP12.2, JP13.2, JP14.2, JP15.2, JP16.2, JP2.2, JP3.2, JP5.2, JP6.2, JP7.2, JP8.2, JP9.2, U$1.GND, U$1.~G2A, U$2.GND, U$2.~G2A, U$3.GND, U1.PD3(INT1); no longer C2.2, C9.-, R1.1, R2.1, TLC5947-2.GND, TLC5947.GND, U1.PB0(ICP), U1.PC4(ADC4/SDA), U1.PD5(T1), U1.PD6(AIN0), U1.PD7(AIN1)
- net N$1: now also JP1.1; no longer R1.2, TLC5947.IREF
- net N$14: now also JP4.1; no longer 1.2, TLC5947.OUT1
- net N$2: now also JP2.1; no longer R2.2, TLC5947-2.IREF
- net N$9: now also JP3.1; no longer 1.1, TLC5947.OUT2
- net NC: no longer U$18.5
- net VCC: now also C9.1, U$1.VCC, U$2.VCC, U$3.VCC; no longer C2.1, JP4.1, TLC5947-2.VCC, TLC5947.VCC
- net VDD: now also C2.+, JP1.4, JP10.4, JP11.4, JP12.4, JP13.4, JP14.4, JP15.4, JP16.4, JP2.4, JP3.4, JP4.4, JP5.4, JP6.4, JP7.4, JP8.4, JP9.4; no longer 1.4, 10.4, 11.4, 12.4, 13.4, 14.4, 15.4, 16.4, 2.4, 3.4, 4.4, 5.4, 6.4, 7.4, 8.4, 9.4, C9.+
Other:
- moved on the sheet: C1, F1, J1, LED2, R5, U$18, U$21
