File: ATTINY_WS2812.sch (EAGLE design)
At the start: 33 parts, among them J1 POWER_JACKPTH, U2 ATTINY2313A, Y1 16MHZ

Commit message: attiny2313 control board
Parts:
- removed C8: 10uF, SparkFun:CAP_POL1206
- removed MIC5205: ###V, SparkFun:V_REG_LDOSMD
Connections:
- removed net DI: JP1.3
- removed net N$5: U$21.1, U$21.2, U$21.3, U$21.4
- removed net PB0: U$21.5, U2.PB0
- removed net PB1: U$21.6, U2.PB1
- removed net PB2: U$21.7, U2.PB2
- removed net PB3: U$21.8, U2.PB3
- removed net VDD: C2.+, C8.+, F1.2, JP1.4, JP10.4, JP2.4, JP3.4, JP4.4, JP5.4, JP6.4, JP7.4, JP8.4, JP9.4, MIC5205.EN, MIC5205.IN
- new net N$1: U$21.5, U2.PB3
- new net N$3: U$21.6, U2.PB2
- new net N$6: U$21.7, U2.PB1
- new net N$9: U$21.8, U2.PB0
- net GND: now also U$21.1, U$21.2, U$21.3, U$21.4; no longer C8.-, MIC5205.GND
- net VCC: now also C2.+, F1.2, JP1.4, JP10.4, JP2.4, JP3.4, JP4.4, JP5.4, JP6.4, JP7.4, JP8.4, JP9.4; no longer MIC5205.OUT
- net WS: now also JP1.3
Other:
- moved on the sheet: C2, C3, U$21
