File: schematics/ATTINY_WS2812.brd (EAGLE design)
At the start: 58.4 x 38.1 mm, 34 parts, among them J1 POWER_JACKPTH, U2 ATTINY2313A, Y1 16MHZ

Commit message: changed WS2812 controller to uUSB, minor spacing edits to everything else
Changed lines of the file:
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@@
 <text x="39.243" y="30.099" size="0.8128" layer="25" distance="130" rot="R270">VCC MOSI GND
 MISO SCK RST</text>
+<circle x="2.667" y="32.385" radius="2.54" width="0.4064" layer="21"/>
 </plain>
 <attributes>
