File: schematics/dmx_splitter.sch (EAGLE design)
At the start: 81 parts

Commit message: Made DMX splitter board for RPi -> other boards. iff --git a/schematics/dmx_splitter.brd b/schematics/dmx_splitter.brd new file mode 100644 index 0000000..f48532d --- /dev/null +++ b/schematics/dmx_splitter.brd @@ -0,0 +1,1127 @@ +<?xml version="1.0" encoding="utf-8"?> +<!DOCTYPE eagle SYSTEM "eagle.dtd"> +<eagle version="6.4"> +<drawing> +<settings> +<setting alwaysvectorfont="yes"/> +<setting verticaltext="up"/> +</settings> +<grid distance="0.01" unitdist="inch" unit="inch" style="lines" multiple="1" display="yes" altdistance="0.025" altunitdist="inch" altunit="inch"/> +<layers> +<layer number="1" name="Top" color="4" fill="1" visible="yes" active="yes"/> +<layer number="16" name="Bottom" color="1" fill="1" visible="yes" active="yes"/> +<layer number="17" name="Pads" color="2" fill="1" visible="yes" active="yes"/> +<layer number="18" name="Vias" color="2" fill="1" visible="yes" active="yes"/> +<layer number="19" name="Unrouted" color="6" fill="1" visible="yes" active="yes"/> +<layer number="20" name="Dimension" color="15" fill="1" visible="yes" active="yes"/> +<layer number="21" name="tPlace" color="7" fill="1" visible="yes" active="yes"/> +<layer number="22" name="bPlace" color="7" fill="1" visible="yes" active="yes"/> +<layer number="23" name="tOrigins" color="15" fill="1" visible="yes" active="yes"/> +<layer number="24" name="bOrigins" color="15" fill="1" visible="yes" active="yes"/> +<layer number="25" name="tNames" color="7" fill="1" visible="yes" active="yes"/> +<layer number="26" name="bNames" color="7" fill="1" visible="yes" active="yes"/> +<layer number="27" name="tValues" color="7" fill="1" visible="yes" active="yes"/> +<layer number="28" name="bValues" color="7" fill="1" visible="yes" active="yes"/> +<layer number="29" name="tStop" color="7" fill="3" visible="no" active="yes"/> +<layer number="30" name="bStop" color="7" fill="6" visible="no" active="yes"/> +<layer number="31" name="tCream" color="7" fill="4" visible="no" active="yes"/> +<layer number="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
Parts:
- removed C13, C14, C16, C17, C18, C19, C20: .1uF, SparkFun-Capacitors:CAP0402-CAP
- removed E13, E14, E15, E16, E17, E18, E19, E20: RJ45-8PTH, SparkFun-Connectors:RJ45-8PTH
- removed R10, R11, R12, R13, R14, R15, R16, R17, R18, R19, R2, R20, R3, R4, R5, R6, R7, R8, R9: 100, SparkFun-Passives:RESISTOR1206
- removed S13, S14, S15, S16, S17, S18, S19, S20: 75176B, 751xx:75176B
- removed U$1: RASPBERRY-PI_REV1, RaspberryPi:RASPBERRY-PI_REV1
- added JP1: USB-MICROB, SparkFun-Connectors:USB-MICROB
Connections:
- removed net DATA1+_10: E10.1, R10.1, S10.A
- removed net DATA1+_15: E15.1, R15.1, S15.A
- removed net DATA1+_16: E16.1, R16.1, S16.A
- removed net DATA1+_17: E17.1, R17.1, S17.A
- removed net DATA1+_18: E18.1, R18.1, S18.A
- removed net DATA1+_19: E19.1, R19.1, S19.A
- removed net DATA1+_20: E20.1, R20.1, S20.A
- removed net DATA1+_9: E9.1, R9.1, S9.A
- removed net DATA1-_10: E10.2, R10.2, S10.B
- removed net DATA1-_15: E15.2, R15.2, S15.B
- removed net DATA1-_16: E16.2, R16.2, S16.B
- removed net DATA1-_17: E17.2, R17.2, S17.B
- removed net DATA1-_18: E18.2, R18.2, S18.B
- removed net DATA1-_19: E19.2, R19.2, S19.B
- removed net DATA1-_20: E20.2, R20.2, S20.B
- removed net DATA1-_9: E9.2, R9.2, S9.B
- removed net DATA2+_10: E10.3
- removed net DATA2+_15: E15.3
- removed net DATA2+_16: E16.3
- removed net DATA2+_17: E17.3
- removed net DATA2+_18: E18.3
- removed net DATA2+_19: E19.3
- removed net DATA2+_20: E20.3
- removed net DATA2+_9: E9.3
- removed net DATA2-_10: E10.6
- removed net DATA2-_15: E15.6
- removed net DATA2-_16: E16.6
- removed net DATA2-_17: E17.6
- removed net DATA2-_18: E18.6
- removed net DATA2-_19: E19.6
- removed net DATA2-_20: E20.6
- removed net DATA2-_9: E9.6
- removed net RE/DE: S1.!RE, S1.DE, S10.!RE, S10.DE, S11.!RE, S11.DE, S12.!RE, S12.DE, S13.!RE, S13.DE, S14.!RE, S14.DE, S15.!RE, S15.DE, S16.!RE, S16.DE, S17.!RE, S17.DE, S18.!RE, S18.DE, S19.!RE, S19.DE, S2.!RE, S2.DE, S20.!RE, S20.DE, S3.!RE, S3.DE, S4.!RE, S4.DE, S5.!RE, S5.DE, S6.!RE, S6.DE, S7.!RE, S7.DE, S8.!RE, S8.DE, S9.!RE, S9.DE, U$1.GPIO17
- removed net RXI: S1.R, S10.R, S11.R, S12.R, S13.R, S14.R, S15.R, S16.R, S17.R, S18.R, S19.R, S2.R, S20.R, S3.R, S4.R, S5.R, S6.R, S7.R, S8.R, S9.R, U$1.GPIO15,UART0_RXD
- net DATA1+_11: now also E9.1, S9.A; no longer E11.1, R11.1, S11.A
- net DATA1+_12: now also E10.1, S10.A; no longer E12.1, R12.1, S12.A
- net DATA1+_13: now also E11.1, S11.A; no longer E13.1, R13.1, S13.A
- net DATA1+_14: now also E12.1, S12.A; no longer E14.1, R14.1, S14.A
- net DATA1+_2: no longer R2.1
- net DATA1+_3: no longer R3.1
- net DATA1+_4: no longer R4.1
- net DATA1+_5: no longer R5.1
- net DATA1+_6: no longer R6.1
- net DATA1+_7: no longer R7.1
- net DATA1+_8: no longer R8.1
- net DATA1-_11: now also E9.2, S9.B; no longer E11.2, R11.2, S11.B
- net DATA1-_12: now also E10.2, S10.B; no longer E12.2, R12.2, S12.B
- net DATA1-_13: now also E11.2, S11.B; no longer E13.2, R13.2, S13.B
- net DATA1-_14: now also E12.2, S12.B; no longer E14.2, R14.2, S14.B
- net DATA1-_2: no longer R2.2
- net DATA1-_3: no longer R3.2
- net DATA1-_4: no longer R4.2
- net DATA1-_5: no longer R5.2
- net DATA1-_6: no longer R6.2
- net DATA1-_7: no longer R7.2
- net DATA1-_8: no longer R8.2
- net DATA2+_11: now also E9.3; no longer E11.3
- net DATA2+_12: now also E10.3; no longer E12.3
- net DATA2+_13: now also E11.3; no longer E13.3
- net DATA2+_14: now also E12.3; no longer E14.3
- net DATA2-_11: now also E9.6; no longer E11.6
- net DATA2-_12: now also E10.6; no longer E12.6
- net DATA2-_13: now also E11.6; no longer E13.6
- net DATA2-_14: now also E12.6; no longer E14.6
- net GND: now also JP1.GND, S1.!RE, S1.D, S1.DE; no longer C13.2, C14.2, C16.2, C17.2, C18.2, C19.2, C20.2, E13.7, E13.8, E14.7, E14.8, E15.7, E15.8, E16.7, E16.8, E17.7, E17.8, E18.7, E18.8, E19.7, E19.8, E20.7, E20.8, S13.GND, S14.GND, S15.GND, S16.GND, S17.GND, S18.GND, S19.GND, S20.GND, U$1.GND@14, U$1.GND@20, U$1.GND@25, U$1.GND@6, U$1.GND@9
- net TXO: now also S1.R; no longer S1.D, S13.D, S14.D, S15.D, S16.D, S17.D, S18.D, S19.D, S20.D, U$1.GPIO14,UART0_TXD
- net VCC: now also JP1.VBUS, S10.!RE, S10.DE, S11.!RE, S11.DE, S12.!RE, S12.DE, S2.!RE, S2.DE, S3.!RE, S3.DE, S4.!RE, S4.DE, S5.!RE, S5.DE, S6.!RE, S6.DE, S7.!RE, S7.DE, S8.!RE, S8.DE, S9.!RE, S9.DE; no longer C13.1, C14.1, C16.1, C17.1, C18.1, C19.1, C20.1, S13.VCC, S14.VCC, S15.VCC, S16.VCC, S17.VCC, S18.VCC, S19.VCC, S20.VCC, U$1.5V@2
Other:
- moved on the sheet: C10, C11, C12, C15, C9, E10, E11, E12, E9, S10, S11, S12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
